Commit message: delete property

File: simrobo_description/urdf/wheel/wheel.urdf.xacro (robot description, xacro)
@@ -2,7 +2,4 @@
 <robot name="wheel" xmlns:xacro="http://www.ros.org/wiki/xacro">
   <xacro:macro name="wheel" params="name parent radius clearance mass *origin">
-    <xacro:property name="WHEEL_RADIUS" value="0.14"/>
-    <xacro:property name="WHEEL_CLEARANCE" value="0.01"/>
-    <xacro:property name="WHEEL_MASS" value="0.4"/>
     <material name="${name}_wheel_color">
       <color rgba="0.0 0.0 1.0 1.0"/>
