Commit message: change tags from property to params

File: simrobo_description/urdf/body/body.urdf.xacro (robot description, xacro)
@@ -1,21 +1,17 @@
 <?xml version="1.0" ?>
 <robot name="body" xmlns:xacro="http://www.ros.org/wiki/xacro">
-  <xacro:macro name="body" params="name *origin">
-    <xacro:property name="BODY_DEPTH" value="0.14"/>
-    <xacro:property name="BODY_WIDTH" value="0.1"/>
-    <xacro:property name="BODY_HEIGHT" value="0.2"/>
-    <xacro:property name="MASS" value="1"/>
+  <xacro:macro name="body" params="name depth width height mass *origin">
     <link name="${name}">
       <inertial>
         <origin xyz="0 0 0" rpy="0 0 0"/>
-        <mass value="${MASS}" />
-        <inertia ixx="${MASS/12*(BODY_WIDTH*BODY_WIDTH+BODY_HEIGHT*BODY_HEIGHT)}" ixy="0" ixz="0"
-                 iyx="0" iyy="${MASS/12*(BODY_DEPTH*BODY_DEPTH+BODY_HEIGHT*BODY_HEIGHT)}" iyz="0"
-                 izx="0" izy="0" izz="${MASS/12*(BODY_DEPTH*BODY_DEPTH+BODY_WIDTH*BODY_WIDTH)}"/>
+        <mass value="${mass}" />
+        <inertia ixx="${mass/12*(width*width+height*height)}" ixy="0" ixz="0"
+                 iyx="0" iyy="${mass/12*(depth*depth+height*height)}" iyz="0"
+                 izx="0" izy="0" izz="${mass/12*(depth*depth+width*width)}"/>
       </inertial>
       <visual>
-        <origin xyz="0 0 ${BODY_HEIGHT/2}" rpy="0 0 0"/>
+        <origin xyz="0 0 ${height/2}" rpy="0 0 0"/>
         <geometry>
-          <box size="${BODY_DEPTH} ${BODY_WIDTH} ${BODY_HEIGHT}"/>
+          <box size="${depth} ${width} ${height}"/>
         </geometry>
         <material name="body_color">
@@ -24,7 +20,7 @@
       </visual>
       <collision>
-        <origin xyz="0 0 ${BODY_HEIGHT/2}" rpy="0 0 0"/>
+        <origin xyz="0 0 ${height/2}" rpy="0 0 0"/>
         <geometry>
-          <box size="${BODY_DEPTH} ${BODY_WIDTH} ${BODY_HEIGHT}"/>
+          <box size="${depth} ${width} ${height}"/>
         </geometry>
       </collision>

File: simrobo_description/urdf/simrobo.urdf.xacro (robot description, xacro)
@@ -5,4 +5,8 @@
   <xacro:include filename="$(find simrobo_description)/urdf/wheel/wheel.urdf.xacro" />
   <!-- property -->
+  <xacro:property name="body_depth" value="0.14"/>
+  <xacro:property name="body_width" value="0.1"/>
+  <xacro:property name="body_height" value="0.2"/>
+  <xacro:property name="body_mass" value="1"/>
   <xacro:property name="wheel_radius" value="0.14"/>
   <xacro:property name="wheel_clearance" value="0.01"/>
@@ -10,5 +14,5 @@
   <!-- ======== Body Description ======== -->
   <link name="base_footprint"/>
-  <xacro:body name="base_link">
+  <xacro:body name="base_link" depth="${body_depth}" width="${body_width}" height="${body_height}" mass="${body_mass}">
     <origin xyz="0 0 0" rpy="0 0 0"/>
   </xacro:body>

Commit message: add body color

File: simrobo_description/urdf/body/body.urdf.xacro (robot description, xacro)
@@ -27,4 +27,5 @@
     </link>
     <gazebo reference="${name}">
+      <material>Gazebo/Yellow</material>
       <mu1 value="0.8"/>
       <mu2 value="0.8"/>
