Commit message: add wheel

File: simrobo_description/urdf/simrobo.urdf.xacro (robot description, xacro)
@@ -3,4 +3,9 @@
   <!-- include xacro files -->
   <xacro:include filename="$(find simrobo_description)/urdf/body/body.urdf.xacro" />
+  <xacro:include filename="$(find simrobo_description)/urdf/wheel/wheel.urdf.xacro" />
+  <!-- property -->
+  <xacro:property name="wheel_radius" value="0.14"/>
+  <xacro:property name="wheel_clearance" value="0.01"/>
+  <xacro:property name="wheel_mass" value="0.4"/>
   <!-- ======== Body Description ======== -->
   <link name="base_footprint"/>
@@ -8,3 +13,10 @@
     <origin xyz="0 0 0" rpy="0 0 0"/>
   </xacro:body>
+  <!-- ======== Wheel Description ======== -->
+  <xacro:wheel name="left" parent="base_link" radius="${wheel_radius}" clearance="${wheel_clearance}" mass="${wheel_mass}">
+    <origin xyz="1 0 0" rpy="0 0 0"/>
+  </xacro:wheel>
+  <xacro:wheel name="right" parent="base_link"  radius="${wheel_radius}" clearance="${wheel_clearance}" mass="${wheel_mass}">
+    <origin xyz="-1 0 0" rpy="0 0 0"/>
+  </xacro:wheel>
 </robot>

Commit message: add joint_state_publisher_gui

File: simrobo_description/urdf/simrobo.urdf.xacro (robot description, xacro)
@@ -9,5 +9,5 @@
   <xacro:property name="body_height" value="0.2"/>
   <xacro:property name="body_mass" value="1"/>
-  <xacro:property name="wheel_radius" value="0.14"/>
+  <xacro:property name="wheel_radius" value="0.1"/>
   <xacro:property name="wheel_clearance" value="0.01"/>
   <xacro:property name="wheel_mass" value="0.4"/>
@@ -19,8 +19,8 @@
   <!-- ======== Wheel Description ======== -->
   <xacro:wheel name="left" parent="base_link" radius="${wheel_radius}" clearance="${wheel_clearance}" mass="${wheel_mass}">
-    <origin xyz="1 0 0" rpy="0 0 0"/>
+    <origin xyz="0 ${body_width/2} 0" rpy="${-pi/2} 0 0"/>
   </xacro:wheel>
   <xacro:wheel name="right" parent="base_link"  radius="${wheel_radius}" clearance="${wheel_clearance}" mass="${wheel_mass}">
-    <origin xyz="-1 0 0" rpy="0 0 0"/>
+    <origin xyz="0 ${-body_width/2} 0" rpy="${-pi/2} 0 0"/>
   </xacro:wheel>
 </robot>

File: simrobo_description/urdf/wheel/wheel.urdf.xacro (robot description, xacro)
@@ -27,9 +27,9 @@
       </collision>
     </link>
-    <joint name="${name}_wheel_joint" type="fixed">
+    <joint name="${name}_wheel_joint" type="continuous">
       <xacro:insert_block name="origin"/>
       <parent link="${parent}"/>
       <child link="${name}_wheel_link"/>
-      <axis xyz="0 0 1"/>
+      <axis xyz="0.0 0.0 1.0"/>
     </joint>
   </xacro:macro>

Commit message: fix joint origin

File: simrobo_description/urdf/simrobo.urdf.xacro (robot description, xacro)
@@ -15,12 +15,12 @@
   <link name="base_footprint"/>
   <xacro:body name="base_link" depth="${body_depth}" width="${body_width}" height="${body_height}" mass="${body_mass}">
-    <origin xyz="0 0 0" rpy="0 0 0"/>
+    <origin xyz="0 0 ${wheel_radius}" rpy="0 0 0"/>
   </xacro:body>
   <!-- ======== Wheel Description ======== -->
   <xacro:wheel name="left" parent="base_link" radius="${wheel_radius}" clearance="${wheel_clearance}" mass="${wheel_mass}">
-    <origin xyz="0 ${body_width/2} 0" rpy="${-pi/2} 0 0"/>
+    <origin xyz="0 ${body_width/2+wheel_clearance/2} 0" rpy="${-pi/2} 0 0"/>
   </xacro:wheel>
   <xacro:wheel name="right" parent="base_link"  radius="${wheel_radius}" clearance="${wheel_clearance}" mass="${wheel_mass}">
-    <origin xyz="0 ${-body_width/2} 0" rpy="${-pi/2} 0 0"/>
+    <origin xyz="0 ${-body_width/2-wheel_clearance/2} 0" rpy="${-pi/2} 0 0"/>
   </xacro:wheel>
 </robot>

Commit message: add caster

File: simrobo_description/urdf/simrobo.urdf.xacro (robot description, xacro)
@@ -4,4 +4,5 @@
   <xacro:include filename="$(find simrobo_description)/urdf/body/body.urdf.xacro" />
   <xacro:include filename="$(find simrobo_description)/urdf/wheel/wheel.urdf.xacro" />
+  <xacro:include filename="$(find simrobo_description)/urdf/wheel/caster.urdf.xacro" />
   <!-- property -->
   <xacro:property name="body_depth" value="0.14"/>
@@ -12,4 +13,6 @@
   <xacro:property name="wheel_clearance" value="0.01"/>
   <xacro:property name="wheel_mass" value="0.4"/>
+  <xacro:property name="caster_radius" value="0.04"/>
+  <xacro:property name="caster_mass" value="0.2"/>
   <!-- ======== Body Description ======== -->
   <link name="base_footprint"/>
@@ -21,6 +24,9 @@
     <origin xyz="0 ${body_width/2+wheel_clearance/2} 0" rpy="${-pi/2} 0 0"/>
   </xacro:wheel>
-  <xacro:wheel name="right" parent="base_link"  radius="${wheel_radius}" clearance="${wheel_clearance}" mass="${wheel_mass}">
+  <xacro:wheel name="right" parent="base_link" radius="${wheel_radius}" clearance="${wheel_clearance}" mass="${wheel_mass}">
     <origin xyz="0 ${-body_width/2-wheel_clearance/2} 0" rpy="${-pi/2} 0 0"/>
   </xacro:wheel>
+  <xacro:caster name="back" parent="base_link" radius="${caster_radius}" mass="${caster_mass}">
+    <origin xyz="0 0 ${-wheel_radius+caster_radius}" rpy="0 0 0"/>
+  </xacro:caster>
 </robot>

Commit message: add properties

File: simrobo_description/urdf/simrobo.urdf.xacro (robot description, xacro)
@@ -13,6 +13,8 @@
   <xacro:property name="wheel_clearance" value="0.01"/>
   <xacro:property name="wheel_mass" value="0.4"/>
+  <xacro:property name="wheel_joint_x" value="0.1"/>
   <xacro:property name="caster_radius" value="0.04"/>
   <xacro:property name="caster_mass" value="0.2"/>
+  <xacro:property name="caster_joint_x" value="-0.1"/>
   <!-- ======== Body Description ======== -->
   <link name="base_footprint"/>
@@ -22,11 +24,11 @@
   <!-- ======== Wheel Description ======== -->
   <xacro:wheel name="left" parent="base_link" radius="${wheel_radius}" clearance="${wheel_clearance}" mass="${wheel_mass}">
-    <origin xyz="0 ${body_width/2+wheel_clearance/2} 0" rpy="${-pi/2} 0 0"/>
+    <origin xyz="${wheel_joint_x} ${body_width/2+wheel_clearance/2} 0" rpy="${-pi/2} 0 0"/>
   </xacro:wheel>
   <xacro:wheel name="right" parent="base_link" radius="${wheel_radius}" clearance="${wheel_clearance}" mass="${wheel_mass}">
-    <origin xyz="0 ${-body_width/2-wheel_clearance/2} 0" rpy="${-pi/2} 0 0"/>
+    <origin xyz="${wheel_joint_x} ${-body_width/2-wheel_clearance/2} 0" rpy="${-pi/2} 0 0"/>
   </xacro:wheel>
   <xacro:caster name="back" parent="base_link" radius="${caster_radius}" mass="${caster_mass}">
-    <origin xyz="0 0 ${-wheel_radius+caster_radius}" rpy="0 0 0"/>
+    <origin xyz="${caster_joint_x} 0 ${-wheel_radius+caster_radius}" rpy="0 0 0"/>
   </xacro:caster>
 </robot>

Commit message: change property value

File: simrobo_description/urdf/simrobo.urdf.xacro (robot description, xacro)
@@ -6,6 +6,6 @@
   <xacro:include filename="$(find simrobo_description)/urdf/wheel/caster.urdf.xacro" />
   <!-- property -->
-  <xacro:property name="body_depth" value="0.14"/>
-  <xacro:property name="body_width" value="0.1"/>
+  <xacro:property name="body_depth" value="0.4"/>
+  <xacro:property name="body_width" value="0.3"/>
   <xacro:property name="body_height" value="0.2"/>
   <xacro:property name="body_mass" value="1"/>
@@ -13,8 +13,8 @@
   <xacro:property name="wheel_clearance" value="0.01"/>
   <xacro:property name="wheel_mass" value="0.4"/>
-  <xacro:property name="wheel_joint_x" value="0.1"/>
-  <xacro:property name="caster_radius" value="0.04"/>
+  <xacro:property name="wheel_joint_x" value="-0.1"/>
+  <xacro:property name="caster_radius" value="0.08"/>
   <xacro:property name="caster_mass" value="0.2"/>
-  <xacro:property name="caster_joint_x" value="-0.1"/>
+  <xacro:property name="caster_joint_x" value="0.1"/>
   <!-- ======== Body Description ======== -->
   <link name="base_footprint"/>
@@ -29,5 +29,5 @@
     <origin xyz="${wheel_joint_x} ${-body_width/2-wheel_clearance/2} 0" rpy="${-pi/2} 0 0"/>
   </xacro:wheel>
-  <xacro:caster name="back" parent="base_link" radius="${caster_radius}" mass="${caster_mass}">
+  <xacro:caster name="front" parent="base_link" radius="${caster_radius}" mass="${caster_mass}">
     <origin xyz="${caster_joint_x} 0 ${-wheel_radius+caster_radius}" rpy="0 0 0"/>
   </xacro:caster>

Commit message: change wheel clearance

File: simrobo_description/urdf/simrobo.urdf.xacro (robot description, xacro)
@@ -11,5 +11,5 @@
   <xacro:property name="body_mass" value="1"/>
   <xacro:property name="wheel_radius" value="0.1"/>
-  <xacro:property name="wheel_clearance" value="0.01"/>
+  <xacro:property name="wheel_clearance" value="0.03"/>
   <xacro:property name="wheel_mass" value="0.4"/>
   <xacro:property name="wheel_joint_x" value="-0.1"/>

Commit message: add lidar

File: simrobo_description/urdf/simrobo.urdf.xacro (robot description, xacro)
@@ -5,4 +5,5 @@
   <xacro:include filename="$(find simrobo_description)/urdf/wheel/wheel.urdf.xacro" />
   <xacro:include filename="$(find simrobo_description)/urdf/wheel/caster.urdf.xacro" />
+  <xacro:include filename="$(find simrobo_description)/urdf/sensors/lidar.urdf.xacro" />
   <!-- property -->
   <xacro:property name="body_depth" value="0.4"/>
@@ -17,4 +18,7 @@
   <xacro:property name="caster_mass" value="0.2"/>
   <xacro:property name="caster_joint_x" value="0.1"/>
+  <xacro:property name="lidar_radius" value="0.04"/>
+  <xacro:property name="lidar_length" value="0.04"/>
+  <xacro:property name="lidar_mass" value="0.015"/>
   <!-- ======== Body Description ======== -->
   <link name="base_footprint"/>
@@ -32,3 +36,7 @@
     <origin xyz="${caster_joint_x} 0 ${-wheel_radius+caster_radius}" rpy="0 0 0"/>
   </xacro:caster>
+  <!-- ======== Sensors Description ======== -->
+  <xacro:lidar name="laser" parent="base_link" radius="${lidar_radius}" length="${lidar_length}" mass="${lidar_mass}">
+    <origin xyz="0 0 ${body_height+lidar_length/2}" rpy="0 0 0"/>
+  </xacro:lidar>
 </robot>

Commit message: add imu

File: simrobo_description/urdf/simrobo.urdf.xacro (robot description, xacro)
@@ -6,4 +6,5 @@
   <xacro:include filename="$(find simrobo_description)/urdf/wheel/caster.urdf.xacro" />
   <xacro:include filename="$(find simrobo_description)/urdf/sensors/lidar.urdf.xacro" />
+  <xacro:include filename="$(find simrobo_description)/urdf/sensors/imu.urdf.xacro" />
   <xacro:include filename="$(find simrobo_description)/urdf/simrobo.ros2_control.xacro" />
   <!-- property -->
@@ -22,4 +23,7 @@
   <xacro:property name="lidar_length" value="0.04"/>
   <xacro:property name="lidar_mass" value="0.015"/>
+  <xacro:property name="imu_length" value="0.02"/>
+  <xacro:property name="imu_height" value="0.01"/>
+  <xacro:property name="imu_mass" value="0.01"/>
   <!-- ======== Body Description ======== -->
   <link name="base_footprint"/>
@@ -41,4 +45,7 @@
     <origin xyz="0 0 ${body_height+lidar_length/2}" rpy="0 0 0"/>
   </xacro:lidar>
+  <xacro:imu name="imu" parent="base_link" length="${imu_length}" height="${imu_height}" mass="${imu_mass}">
+    <origin xyz="0 0 ${body_height/2}" rpy="0 0 0"/>
+  </xacro:imu>
   <!-- ======== ros2_control ======== -->
   <xacro:simrobo_ros2_control name="simrobo"/>

Commit message: add gps

File: simrobo_description/urdf/simrobo.urdf.xacro (robot description, xacro)
@@ -7,4 +7,5 @@
   <xacro:include filename="$(find simrobo_description)/urdf/sensors/lidar.urdf.xacro" />
   <xacro:include filename="$(find simrobo_description)/urdf/sensors/imu.urdf.xacro" />
+  <xacro:include filename="$(find simrobo_description)/urdf/sensors/gps.urdf.xacro" />
   <xacro:include filename="$(find simrobo_description)/urdf/simrobo.ros2_control.xacro" />
   <!-- property -->
@@ -26,4 +27,7 @@
   <xacro:property name="imu_height" value="0.01"/>
   <xacro:property name="imu_mass" value="0.01"/>
+  <xacro:property name="gps_length" value="0.02"/>
+  <xacro:property name="gps_height" value="0.01"/>
+  <xacro:property name="gps_mass" value="0.01"/>
   <!-- ======== Body Description ======== -->
   <link name="base_footprint"/>
@@ -48,4 +52,7 @@
     <origin xyz="0 0 ${body_height/2}" rpy="0 0 0"/>
   </xacro:imu>
+  <xacro:gps name="gps" parent="base_link" length="${gps_length}" height="${gps_height}" mass="${gps_mass}">
+    <origin xyz="0 0 ${body_height/3}" rpy="0 0 0"/>
+  </xacro:gps>
   <!-- ======== ros2_control ======== -->
   <xacro:simrobo_ros2_control name="simrobo"/>

Commit message: add camera

File: simrobo_description/urdf/simrobo.urdf.xacro (robot description, xacro)
@@ -8,4 +8,5 @@
   <xacro:include filename="$(find simrobo_description)/urdf/sensors/imu.urdf.xacro" />
   <xacro:include filename="$(find simrobo_description)/urdf/sensors/gps.urdf.xacro" />
+  <xacro:include filename="$(find simrobo_description)/urdf/sensors/camera.urdf.xacro" />
   <xacro:include filename="$(find simrobo_description)/urdf/simrobo.ros2_control.xacro" />
   <!-- property -->
@@ -30,4 +31,9 @@
   <xacro:property name="gps_height" value="0.01"/>
   <xacro:property name="gps_mass" value="0.01"/>
+  <xacro:property name="camera_depth" value="0.02"/>
+  <xacro:property name="camera_width" value="0.12"/>
+  <xacro:property name="camera_height" value="0.02"/>
+  <xacro:property name="camera_mass" value="0.1"/>
+  <xacro:property name="camera_pos_z" value="0.15"/>
   <!-- ======== Body Description ======== -->
   <link name="base_footprint"/>
@@ -55,4 +61,7 @@
     <origin xyz="0 0 ${body_height/3}" rpy="0 0 0"/>
   </xacro:gps>
+  <xacro:camera name="camera" parent="base_link" depth="${camera_depth}" width="${camera_width}" height="${camera_height}" mass="${camera_mass}">
+    <origin xyz="${(body_depth+camera_depth)/2} 0 ${camera_pos_z}" rpy="0 0 0"/>
+  </xacro:camera>
   <!-- ======== ros2_control ======== -->
   <xacro:simrobo_ros2_control name="simrobo"/>
