Commit message: add use_gpu parameter

File: simrobo_description/urdf/sensors/lidar.gazebo.xacro (robot description, xacro)
@@ -1,38 +1,74 @@
 <?xml version="1.0"?>
 <robot xmlns:xacro="http://www.ros.org/wiki/xacro">
-  <xacro:macro name="lidar_gazebo" params="name:=laser">
+  <xacro:macro name="lidar_gazebo" params="name:=laser gpu:=false">
     <gazebo reference="${name}">
-      <sensor type="ray" name="head_lidar_sensor">
-        <pose>0 0 0 0 0 0</pose>
-        <visualize>true</visualize>
-        <update_rate>20</update_rate>
-        <ray>
-          <scan>
-            <horizontal>
-              <samples>1080</samples>
-              <resolution>1</resolution>
-              <min_angle>${radians(-180)}</min_angle>
-              <max_angle>${radians( 180)}</max_angle>
-            </horizontal>
-          </scan>
-          <range>
-            <min>0.1</min>
-            <max>40.0</max>
-            <resolution>0.01</resolution>
-          </range>
-          <noise>
-            <type>gaussian</type>
-            <mean>0.0</mean>
-            <stddev>0.01</stddev>
-          </noise>
-        </ray>
-        <plugin name="gazebo_ros_head_lidar_controller" filename="libgazebo_ros_ray_sensor.so">
-          <ros>
-            <remapping>~/out:=scan</remapping>
-          </ros>
-          <output_type>sensor_msgs/LaserScan</output_type>
-          <frameName>laser</frameName>
-        </plugin>
-      </sensor>
+      <xacro:if value="${gpu}">
+        <sensor type="gpu_ray" name="head_lidar_sensor">
+          <pose>0 0 0 0 0 0</pose>
+          <visualize>true</visualize>
+          <update_rate>20</update_rate>
+          <ray>
+            <scan>
+              <horizontal>
+                <samples>1080</samples>
+                <resolution>1</resolution>
+                <min_angle>${radians(-180)}</min_angle>
+                <max_angle>${radians( 180)}</max_angle>
+              </horizontal>
+            </scan>
+            <range>
+              <min>0.1</min>
+              <max>40.0</max>
+              <resolution>0.01</resolution>
+            </range>
+            <noise>
+              <type>gaussian</type>
+              <mean>0.0</mean>
+              <stddev>0.01</stddev>
+            </noise>
+          </ray>
+          <plugin name="gazebo_ros_head_lidar_controller" filename="libgazebo_ros_ray_sensor.so">
+            <ros>
+              <remapping>~/out:=scan</remapping>
+            </ros>
+            <output_type>sensor_msgs/LaserScan</output_type>
+            <frameName>laser</frameName>
+          </plugin>
+        </sensor>
+      </xacro:if>
+      <xacro:unless value="${gpu}">
+        <sensor type="ray" name="head_lidar_sensor">
+          <pose>0 0 0 0 0 0</pose>
+          <visualize>true</visualize>
+          <update_rate>20</update_rate>
+          <ray>
+            <scan>
+              <horizontal>
+                <samples>1080</samples>
+                <resolution>1</resolution>
+                <min_angle>${radians(-180)}</min_angle>
+                <max_angle>${radians( 180)}</max_angle>
+              </horizontal>
+            </scan>
+            <range>
+              <min>0.1</min>
+              <max>40.0</max>
+              <resolution>0.01</resolution>
+            </range>
+            <noise>
+              <type>gaussian</type>
+              <mean>0.0</mean>
+              <stddev>0.01</stddev>
+            </noise>
+          </ray>
+          <plugin name="gazebo_ros_head_lidar_controller" filename="libgazebo_ros_ray_sensor.so">
+            <ros>
+              <remapping>~/out:=scan</remapping>
+            </ros>
+            <output_type>sensor_msgs/LaserScan</output_type>
+            <frameName>laser</frameName>
+          </plugin>
+        </sensor>
+      </xacro:unless>
     </gazebo>
   </xacro:macro>

File: simrobo_description/urdf/sensors/lidar.urdf.xacro (robot description, xacro)
@@ -2,5 +2,5 @@
 <robot name="lidar" xmlns:xacro="http://www.ros.org/wiki/xacro">
   <xacro:include filename="$(find simrobo_description)/urdf/sensors/lidar.gazebo.xacro"/>
-  <xacro:macro name="lidar" params="name:=laser parent radius length mass *origin">
+  <xacro:macro name="lidar" params="name:=laser gpu:=false parent radius length mass *origin">
     <material name="${name}_color">
       <color rgba="0.70196 0.70196 0.70196 1.0"/>
@@ -34,5 +34,5 @@
     </joint>
     <!-- Gazebo Plugin -->
-    <xacro:lidar_gazebo name="${name}"/>
+    <xacro:lidar_gazebo name="${name}" gpu="${gpu}"/>
   </xacro:macro>
 </robot>

File: simrobo_description/urdf/sensors/velodyne.gazebo.xacro (robot description, xacro)
@@ -1,46 +1,90 @@
 <?xml version="1.0"?>
 <robot xmlns:xacro="http://www.ros.org/wiki/xacro">
-  <xacro:macro name="velodyne_gazebo" params="name:=velodyne">
+  <xacro:macro name="velodyne_gazebo" params="name:=velodyne gpu:=false">
     <gazebo reference="${name}">
-      <sensor type="ray" name="head_velodyne_sensor">
-        <pose>0 0 0 0 0 0</pose>
-        <visualize>false</visualize>
-        <update_rate>10</update_rate>
-        <ray>
-          <scan>
-            <horizontal>
-              <samples>1024</samples>
-              <resolution>1</resolution>
-              <min_angle>${radians(-180)}</min_angle>
-              <max_angle>${radians( 180)}</max_angle>
-            </horizontal>
-            <vertical>
-              <samples>16</samples>
-              <resolution>1</resolution>
-              <min_angle>${radians(-15)}</min_angle>
-              <max_angle>${radians(15)}</max_angle>
-            </vertical>
-          </scan>
-          <range>
-            <min>0.3</min>
-            <max>101.0</max>
-            <resolution>0.001</resolution>
-          </range>
-          <noise>
-            <type>gaussian</type>
-            <mean>0.0</mean>
-            <stddev>0.0</stddev>
-          </noise>
-        </ray>
-        <plugin name="gazebo_ros_head_velodyne_controller" filename="libgazebo_ros_velodyne_laser.so">
-          <ros>
-            <remapping>~/out:=velodyne_points</remapping>
-          </ros>
-          <frameName>velodyne</frameName>
-          <min_range>0.9</min_range>
-          <max_range>100</max_range>
-          <gaussianNoise>0.008</gaussianNoise>
-        </plugin>
-      </sensor>
+      <xacro:if value="${gpu}">
+        <sensor type="gpu_ray" name="head_velodyne_sensor">
+          <pose>0 0 0 0 0 0</pose>
+          <visualize>false</visualize>
+          <update_rate>10</update_rate>
+          <ray>
+            <scan>
+              <horizontal>
+                <samples>1024</samples>
+                <resolution>1</resolution>
+                <min_angle>${radians(-180)}</min_angle>
+                <max_angle>${radians( 180)}</max_angle>
+              </horizontal>
+              <vertical>
+                <samples>16</samples>
+                <resolution>1</resolution>
+                <min_angle>${radians(-15)}</min_angle>
+                <max_angle>${radians( 15)}</max_angle>
+              </vertical>
+            </scan>
+            <range>
+              <min>0.3</min>
+              <max>101.0</max>
+              <resolution>0.001</resolution>
+            </range>
+            <noise>
+              <type>gaussian</type>
+              <mean>0.0</mean>
+              <stddev>0.0</stddev>
+            </noise>
+          </ray>
+          <plugin name="gazebo_ros_head_velodyne_controller" filename="libgazebo_ros_velodyne_laser.so">
+            <ros>
+              <remapping>~/out:=velodyne_points</remapping>
+            </ros>
+            <frameName>velodyne</frameName>
+            <min_range>0.9</min_range>
+            <max_range>100</max_range>
+            <gaussianNoise>0.008</gaussianNoise>
+          </plugin>
+        </sensor>
+      </xacro:if>
+      <xacro:unless value="${gpu}">
+        <sensor type="ray" name="head_velodyne_sensor">
+          <pose>0 0 0 0 0 0</pose>
+          <visualize>false</visualize>
+          <update_rate>10</update_rate>
+          <ray>
+            <scan>
+              <horizontal>
+                <samples>1024</samples>
+                <resolution>1</resolution>
+                <min_angle>${radians(-180)}</min_angle>
+                <max_angle>${radians( 180)}</max_angle>
+              </horizontal>
+              <vertical>
+                <samples>16</samples>
+                <resolution>1</resolution>
+                <min_angle>${radians(-15)}</min_angle>
+                <max_angle>${radians( 15)}</max_angle>
+              </vertical>
+            </scan>
+            <range>
+              <min>0.3</min>
+              <max>101.0</max>
+              <resolution>0.001</resolution>
+            </range>
+            <noise>
+              <type>gaussian</type>
+              <mean>0.0</mean>
+              <stddev>0.0</stddev>
+            </noise>
+          </ray>
+          <plugin name="gazebo_ros_head_velodyne_controller" filename="libgazebo_ros_velodyne_laser.so">
+            <ros>
+              <remapping>~/out:=velodyne_points</remapping>
+            </ros>
+            <frameName>velodyne</frameName>
+            <min_range>0.9</min_range>
+            <max_range>100</max_range>
+            <gaussianNoise>0.008</gaussianNoise>
+          </plugin>
+        </sensor>
+      </xacro:unless>
     </gazebo>
   </xacro:macro>

File: simrobo_description/urdf/sensors/velodyne.urdf.xacro (robot description, xacro)
@@ -2,5 +2,5 @@
 <robot name="velodyne" xmlns:xacro="http://www.ros.org/wiki/xacro">
   <xacro:include filename="$(find simrobo_description)/urdf/sensors/velodyne.gazebo.xacro"/>
-  <xacro:macro name="velodyne" params="name:=velodyne parent radius length mass *origin">
+  <xacro:macro name="velodyne" params="name:=velodyne gpu:=false parent radius length mass *origin">
     <material name="${name}_color">
       <color rgba="0.70196 0.70196 0.70196 1.0"/>
@@ -34,5 +34,5 @@
     </joint>
     <!-- Gazebo Plugin -->
-    <xacro:velodyne_gazebo name="${name}"/>
+    <xacro:velodyne_gazebo name="${name}" gpu="${gpu}"/>
   </xacro:macro>
 </robot>

File: simrobo_description/urdf/simrobo.urdf.xacro (robot description, xacro)
@@ -6,9 +6,15 @@
   <xacro:include filename="$(find simrobo_description)/urdf/wheel/caster.urdf.xacro" />
   <xacro:include filename="$(find simrobo_description)/urdf/sensors/lidar.urdf.xacro" />
+  <xacro:include filename="$(find simrobo_description)/urdf/sensors/velodyne.urdf.xacro" />
   <xacro:include filename="$(find simrobo_description)/urdf/sensors/imu.urdf.xacro" />
   <xacro:include filename="$(find simrobo_description)/urdf/sensors/gps.urdf.xacro" />
   <xacro:include filename="$(find simrobo_description)/urdf/sensors/camera.urdf.xacro" />
   <xacro:include filename="$(find simrobo_description)/urdf/simrobo.ros2_control.xacro" />
+  <!-- arg -->
+  <xacro:arg name="use_3d_lidar" default="false"/>
+  <xacro:arg name="gpu" default="false"/>
   <!-- property -->
+  <xacro:property name="use_3d_lidar" value="$(arg use_3d_lidar)"/>
+  <xacro:property name="gpu" value="$(arg gpu)"/>
   <xacro:property name="body_depth" value="0.4"/>
   <xacro:property name="body_width" value="0.3"/>
@@ -22,7 +28,11 @@
   <xacro:property name="caster_mass" value="0.2"/>
   <xacro:property name="caster_joint_x" value="0.1"/>
-  <xacro:property name="lidar_radius" value="0.04"/>
-  <xacro:property name="lidar_length" value="0.04"/>
-  <xacro:property name="lidar_mass" value="0.015"/>
+  <xacro:property name="lidar_2d_radius" value="0.04"/>
+  <xacro:property name="lidar_2d_length" value="0.04"/>
+  <xacro:property name="lidar_2d_mass" value="0.015"/>
+  <xacro:property name="lidar_3d_radius" value="0.103"/>
+  <xacro:property name="lidar_3d_length" value="0.0727"/>
+  <xacro:property name="lidar_3d_mass" value="0.830"/>
+  <xacro:property name="lidar_3d_mount_mass" value="0.4"/>
   <xacro:property name="imu_length" value="0.02"/>
   <xacro:property name="imu_height" value="0.01"/>
@@ -52,7 +62,43 @@
   </xacro:caster>
   <!-- ======== Sensors Description ======== -->
-  <xacro:lidar name="laser" parent="base_link" radius="${lidar_radius}" length="${lidar_length}" mass="${lidar_mass}">
-    <origin xyz="0 0 ${body_height+lidar_length/2}" rpy="0 0 0"/>
-  </xacro:lidar>
+  <xacro:if value="${use_3d_lidar}">
+    <link name="lidar_mount">
+      <inertial>
+        <origin xyz="0 0 0" rpy="0 0 0"/>
+        <mass value="${lidar_3d_mount_mass}"/>
+        <inertia ixx="${lidar_3d_mount_mass/12*(3*0.08*0.08+0.3*0.3)}" ixy="0" ixz="0"
+                 iyx="0" iyy="${lidar_3d_mount_mass/12*(3*0.08*0.08+0.3*0.3)}" iyz="0.0"
+                 izx="0" izy="0" izz="${lidar_3d_mount_mass/2*0.08*0.08}"/>
+      </inertial>
+      <visual>
+        <origin xyz="0 0 0" rpy="0 0 0"/>
+        <geometry>
+          <cylinder radius="0.08" length="0.3"/>
+        </geometry>
+        <material name="lidar_mount_color">
+          <color rgba="1.0 1.0 0.0 1.0"/>
+        </material>
+      </visual>
+      <collision>
+        <origin xyz="0 0 0" rpy="0 0 0"/>
+        <geometry>
+          <cylinder  radius="0.08" length="0.3"/>
+        </geometry>
+      </collision>
+    </link>
+    <joint name="lidar_mount_joint" type="fixed">
+      <origin xyz="0 0 ${body_height+0.3/2}" rpy="0 0 0"/>
+      <parent link="base_link"/>
+      <child link="lidar_mount"/>
+    </joint>
+    <xacro:velodyne name="velodyne" gpu="${gpu}" parent="lidar_mount" radius="${lidar_3d_radius}" length="${lidar_3d_length}" mass="${lidar_3d_mass}">
+      <origin xyz="0 0 0.15" rpy="0 0 0"/>
+    </xacro:velodyne>
+  </xacro:if>
+  <xacro:unless value="${use_3d_lidar}">
+    <xacro:lidar name="laser" gpu="${gpu}" parent="base_link" radius="${lidar_2d_radius}" length="${lidar_2d_length}" mass="${lidar_2d_mass}">
+      <origin xyz="0 0 ${body_height+lidar_2d_length/2}" rpy="0 0 0"/>
+    </xacro:lidar>
+  </xacro:unless>
   <xacro:imu name="imu" parent="base_link" length="${imu_length}" height="${imu_height}" mass="${imu_mass}">
     <origin xyz="0 0 ${body_height/2}" rpy="0 0 0"/>
