Commit message: Integrate for ignition

File: simrobo_description/urdf/sensors/lidar.gazebo.xacro (robot description, xacro)
@@ -1,73 +1,111 @@
 <?xml version="1.0"?>
 <robot xmlns:xacro="http://www.ros.org/wiki/xacro">
-  <xacro:macro name="lidar_gazebo" params="name:=laser gpu:=false">
+  <xacro:macro name="lidar_gazebo" params="name:=laser use_ignition:=true gpu:=false">
     <gazebo reference="${name}">
-      <xacro:if value="${gpu}">
-        <sensor type="gpu_ray" name="head_lidar_sensor">
-          <pose>0 0 0 0 0 0</pose>
-          <visualize>true</visualize>
+      <xacro:if value="${use_ignition}">
+        <sensor type="gpu_lidar" name="head_lidar_sensor">
+          <ignition_frame_id>laser</ignition_frame_id>
+          <topic>scan</topic>
           <update_rate>20</update_rate>
-          <ray>
-            <scan>
-              <horizontal>
-                <samples>1080</samples>
-                <resolution>1</resolution>
-                <min_angle>${radians(-180)}</min_angle>
-                <max_angle>${radians( 180)}</max_angle>
-              </horizontal>
-            </scan>
-            <range>
-              <min>0.1</min>
-              <max>40.0</max>
-              <resolution>0.01</resolution>
-            </range>
-            <noise>
-              <type>gaussian</type>
-              <mean>0.0</mean>
-              <stddev>0.01</stddev>
-            </noise>
-          </ray>
-          <plugin name="gazebo_ros_head_lidar_controller" filename="libgazebo_ros_ray_sensor.so">
-            <ros>
-              <remapping>~/out:=scan</remapping>
-            </ros>
-            <output_type>sensor_msgs/LaserScan</output_type>
-            <frameName>laser</frameName>
-          </plugin>
+          <lidar>
+           <scan>
+             <horizontal>
+               <samples>1080</samples>
+               <resolution>1</resolution>
+               <min_angle>${radians(-180)}</min_angle>
+               <max_angle>${radians( 180)}</max_angle>
+             </horizontal>
+             <vertical>
+               <samples>1</samples>
+               <resolution>1</resolution>
+               <min_angle>${radians(-180)}</min_angle>
+               <max_angle>${radians( 180)}</max_angle>
+             </vertical>
+           </scan>
+           <range>
+             <min>0.1</min>
+             <max>40.0</max>
+             <resolution>0.01</resolution>
+           </range>
+           <noise>
+             <type>gaussian</type>
+             <mean>0.0</mean>
+             <stddev>0.01</stddev>
+           </noise>
+           <frame_id>/laser</frame_id>
+         </lidar>
+         <alwaysOn>1</alwaysOn>
+         <visualize>true</visualize>
         </sensor>
       </xacro:if>
-      <xacro:unless value="${gpu}">
-        <sensor type="ray" name="head_lidar_sensor">
-          <pose>0 0 0 0 0 0</pose>
-          <visualize>true</visualize>
-          <update_rate>20</update_rate>
-          <ray>
-            <scan>
-              <horizontal>
-                <samples>1080</samples>
-                <resolution>1</resolution>
-                <min_angle>${radians(-180)}</min_angle>
-                <max_angle>${radians( 180)}</max_angle>
-              </horizontal>
-            </scan>
-            <range>
-              <min>0.1</min>
-              <max>40.0</max>
-              <resolution>0.01</resolution>
-            </range>
-            <noise>
-              <type>gaussian</type>
-              <mean>0.0</mean>
-              <stddev>0.01</stddev>
-            </noise>
-          </ray>
-          <plugin name="gazebo_ros_head_lidar_controller" filename="libgazebo_ros_ray_sensor.so">
-            <ros>
-              <remapping>~/out:=scan</remapping>
-            </ros>
-            <output_type>sensor_msgs/LaserScan</output_type>
-            <frameName>laser</frameName>
-          </plugin>
-        </sensor>
+      <xacro:unless value="${use_ignition}">
+        <xacro:if value="${gpu}">
+          <sensor type="gpu_ray" name="head_lidar_sensor">
+            <pose>0 0 0 0 0 0</pose>
+            <visualize>true</visualize>
+            <update_rate>20</update_rate>
+            <ray>
+              <scan>
+                <horizontal>
+                  <samples>1080</samples>
+                  <resolution>1</resolution>
+                  <min_angle>${radians(-180)}</min_angle>
+                  <max_angle>${radians( 180)}</max_angle>
+                </horizontal>
+              </scan>
+              <range>
+                <min>0.1</min>
+                <max>40.0</max>
+                <resolution>0.01</resolution>
+              </range>
+              <noise>
+                <type>gaussian</type>
+                <mean>0.0</mean>
+                <stddev>0.01</stddev>
+              </noise>
+            </ray>
+            <plugin name="gazebo_ros_head_lidar_controller" filename="libgazebo_ros_ray_sensor.so">
+              <ros>
+                <remapping>~/out:=scan</remapping>
+              </ros>
+              <output_type>sensor_msgs/LaserScan</output_type>
+              <frameName>laser</frameName>
+            </plugin>
+          </sensor>
+        </xacro:if>
+        <xacro:unless value="${gpu}">
+          <sensor type="ray" name="head_lidar_sensor">
+            <pose>0 0 0 0 0 0</pose>
+            <visualize>true</visualize>
+            <update_rate>20</update_rate>
+            <ray>
+              <scan>
+                <horizontal>
+                  <samples>1080</samples>
+                  <resolution>1</resolution>
+                  <min_angle>${radians(-180)}</min_angle>
+                  <max_angle>${radians( 180)}</max_angle>
+                </horizontal>
+              </scan>
+              <range>
+                <min>0.1</min>
+                <max>40.0</max>
+                <resolution>0.01</resolution>
+              </range>
+              <noise>
+                <type>gaussian</type>
+                <mean>0.0</mean>
+                <stddev>0.01</stddev>
+              </noise>
+            </ray>
+            <plugin name="gazebo_ros_head_lidar_controller" filename="libgazebo_ros_ray_sensor.so">
+              <ros>
+                <remapping>~/out:=scan</remapping>
+              </ros>
+              <output_type>sensor_msgs/LaserScan</output_type>
+              <frameName>laser</frameName>
+            </plugin>
+          </sensor>
+        </xacro:unless>
       </xacro:unless>
     </gazebo>

File: simrobo_description/urdf/sensors/lidar.urdf.xacro (robot description, xacro)
@@ -2,5 +2,5 @@
 <robot name="lidar" xmlns:xacro="http://www.ros.org/wiki/xacro">
   <xacro:include filename="$(find simrobo_description)/urdf/sensors/lidar.gazebo.xacro"/>
-  <xacro:macro name="lidar" params="name:=laser gpu:=false parent radius length mass *origin">
+  <xacro:macro name="lidar" params="name:=laser use_ignition:=true gpu:=false parent radius length mass *origin">
     <material name="${name}_color">
       <color rgba="0.70196 0.70196 0.70196 1.0"/>
@@ -34,5 +34,5 @@
     </joint>
     <!-- Gazebo Plugin -->
-    <xacro:lidar_gazebo name="${name}" gpu="${gpu}"/>
+    <xacro:lidar_gazebo name="${name}" use_ignition="${use_ignition}" gpu="${gpu}"/>
   </xacro:macro>
 </robot>

File: simrobo_description/urdf/simrobo.ros2_control.xacro (robot description, xacro)
@@ -1,10 +1,16 @@
 <?xml version="1.0"?>
 <robot xmlns:xacro="http://www.ros.org/wiki/xacro">
-  <xacro:macro name="simrobo_ros2_control" params="name">
+  <xacro:macro name="simrobo_ros2_control" params="name use_ignition">
     <ros2_control name="${name}" type="system">
       <hardware>
-        <plugin>gazebo_ros2_control/GazeboSystem</plugin>
+        <xacro:if value="${use_ignition}">
+          <plugin>gz_ros2_control/GazeboSimSystem</plugin>
+        </xacro:if>
+        <xacro:unless value="${use_ignition}">
+          <plugin>gazebo_ros2_control/GazeboSystem</plugin>
+        </xacro:unless>
       </hardware>
       <joint name="left_wheel_joint">
+        <param name="initial_value">0.0</param>
         <command_interface name="velocity"/>
         <state_interface name="position"/>
@@ -12,4 +18,5 @@
       </joint>
       <joint name="right_wheel_joint">
+        <param name="initial_value">0.0</param>
         <command_interface name="velocity"/>
         <state_interface name="position"/>
@@ -18,7 +25,23 @@
     </ros2_control>
     <gazebo>
-      <plugin filename="libgazebo_ros2_control.so" name="gazebo_ros2_control">
-        <parameters>$(find simrobo_description)/controllers/controllers.yaml</parameters>
-      </plugin>
+      <xacro:if value="${use_ignition}">
+        <plugin
+          filename="ignition-gazebo-sensors-system"
+          name="ignition::gazebo::systems::Sensors">
+          <render_engine>ogre2</render_engine>
+        </plugin>
+        <plugin
+          filename="gz_ros2_control-system"
+          name="gz_ros2_control::GazeboSimROS2ControlPlugin">
+          <robot_param>robot_description</robot_param>
+          <robot_param_node>robot_state_publisher</robot_param_node>
+          <parameters>$(find simrobo_description)/controllers/controllers.yaml</parameters>
+        </plugin>
+      </xacro:if>
+      <xacro:unless value="${use_ignition}">
+        <plugin filename="libgazebo_ros2_control.so" name="gazebo_ros2_control">
+          <parameters>$(find simrobo_description)/controllers/controllers.yaml</parameters>
+        </plugin>
+      </xacro:unless>
     </gazebo>
   </xacro:macro>

File: simrobo_description/urdf/simrobo.urdf.xacro (robot description, xacro)
@@ -7,12 +7,14 @@
   <xacro:include filename="$(find simrobo_description)/urdf/sensors/lidar.urdf.xacro" />
   <xacro:include filename="$(find simrobo_description)/urdf/sensors/velodyne.urdf.xacro" />
-  <xacro:include filename="$(find simrobo_description)/urdf/sensors/imu.urdf.xacro" />
+  <!--xacro:include filename="$(find simrobo_description)/urdf/sensors/imu.urdf.xacro" />
   <xacro:include filename="$(find simrobo_description)/urdf/sensors/gps.urdf.xacro" />
-  <xacro:include filename="$(find simrobo_description)/urdf/sensors/camera.urdf.xacro" />
+  <xacro:include filename="$(find simrobo_description)/urdf/sensors/camera.urdf.xacro" / -->
   <xacro:include filename="$(find simrobo_description)/urdf/simrobo.ros2_control.xacro" />
   <!-- arg -->
+  <xacro:arg name="use_ignition" default="true"/>
   <xacro:arg name="use_3d_lidar" default="false"/>
   <xacro:arg name="gpu" default="false"/>
   <!-- property -->
+  <xacro:property name="use_ignition" value="$(arg use_ignition)"/>
   <xacro:property name="use_3d_lidar" value="$(arg use_3d_lidar)"/>
   <xacro:property name="gpu" value="$(arg gpu)"/>
@@ -97,9 +99,9 @@
   </xacro:if>
   <xacro:unless value="${use_3d_lidar}">
-    <xacro:lidar name="laser" gpu="${gpu}" parent="base_link" radius="${lidar_2d_radius}" length="${lidar_2d_length}" mass="${lidar_2d_mass}">
+    <xacro:lidar name="laser" use_ignition="${use_ignition}" gpu="${gpu}" parent="base_link" radius="${lidar_2d_radius}" length="${lidar_2d_length}" mass="${lidar_2d_mass}">
       <origin xyz="0 0 ${body_height+lidar_2d_length/2}" rpy="0 0 0"/>
     </xacro:lidar>
   </xacro:unless>
-  <xacro:imu name="imu" parent="base_link" length="${imu_length}" height="${imu_height}" mass="${imu_mass}">
+  <!--xacro:imu name="imu" parent="base_link" length="${imu_length}" height="${imu_height}" mass="${imu_mass}">
     <origin xyz="0 0 ${body_height/2}" rpy="0 0 0"/>
   </xacro:imu>
@@ -109,6 +111,6 @@
   <xacro:camera name="camera" parent="base_link" depth="${camera_depth}" width="${camera_width}" height="${camera_height}" mass="${camera_mass}">
     <origin xyz="${(body_depth+camera_depth)/2} 0 ${camera_pos_z}" rpy="0 0 0"/>
-  </xacro:camera>
+  </xacro:camera -->
   <!-- ======== ros2_control ======== -->
-  <xacro:simrobo_ros2_control name="simrobo"/>
+  <xacro:simrobo_ros2_control name="simrobo" use_ignition="${use_ignition}"/>
 </robot>
