Commit message: Add depth camera topic for ignition

File: simrobo_description/urdf/sensors/camera.gazebo.xacro (robot description, xacro)
@@ -1,37 +1,60 @@
 <?xml version="1.0"?>
 <robot xmlns:xacro="http://www.ros.org/wiki/xacro">
-  <xacro:macro name="camera_gazebo" params="name:=camera">
+  <xacro:macro name="camera_gazebo" params="name:=camera use_ignition:=true">
     <gazebo reference="${name}_link">
-      <sensor type="depth" name="${name}">
-        <always_on>true</always_on>
-        <update_rate>15</update_rate>
-        <pose>0 0 0 0 0 0</pose>
-        <!--camera name="${name}">
-          <horizontal_fov>1.46608</horizontal_fov>
-          <image>
-            <width>424</width>
-            <height>240</height>
-            <format>B8G8R8</format>
-          </image>
-          <clip>
-            <near>0.05</near>
-            <far>8</far>
-          </clip>
-        </camera -->
-        <plugin filename="libgazebo_ros_camera.so" name="camera_plugin">
-          <ros>
-            <remapping>camera/image_raw:=color/image_raw</remapping>
-            <remapping>camera/depth/image_raw:=depth_rect_raw</remapping>
-            <remapping>camera/camera_info:=camera_info</remapping>
-            <remapping>camera/depth/camera_info:=depth/camera_info</remapping>
-            <remapping>camera/points:=depth/points</remapping>
-          </ros>
-          <camera_name>${name}</camera_name>
-          <frameName>${name}_link</frameName>
-          <hack_baseline>0.07</hack_baseline>
-          <min_depth>0.05</min_depth>
-          <max_depth>8.0</max_depth>
-        </plugin>
-      </sensor>
+      <xacro:if value="${use_ignition}">
+        <sensor type="depth_camera" name="${name}">
+          <always_on>true</always_on>
+          <update_rate>15</update_rate>
+          <ignition_frame_id>${name}_link</ignition_frame_id>
+          <pose>0 0 0 0 0 0</pose>
+          <camera>
+            <horizontal_fov>1.46608</horizontal_fov>
+            <image>
+              <width>424</width>
+              <height>240</height>
+              <format>R_FLOAT32</format>
+            </image>
+            <clip>
+              <near>0.05</near>
+              <far>8</far>
+            </clip>
+          </camera>
+          <topic>depth_rect_raw</topic>
+        </sensor>
+      </xacro:if>
+      <xacro:unless value="${use_ignition}">
+        <sensor type="depth" name="${name}">
+          <always_on>true</always_on>
+          <update_rate>15</update_rate>
+          <pose>0 0 0 0 0 0</pose>
+          <!--camera name="${name}">
+            <horizontal_fov>1.46608</horizontal_fov>
+            <image>
+              <width>424</width>
+              <height>240</height>
+              <format>B8G8R8</format>
+            </image>
+            <clip>
+              <near>0.05</near>
+              <far>8</far>
+            </clip>
+          </camera -->
+          <plugin filename="libgazebo_ros_camera.so" name="camera_plugin">
+            <ros>
+              <remapping>camera/image_raw:=color/image_raw</remapping>
+              <remapping>camera/depth/image_raw:=depth_rect_raw</remapping>
+              <remapping>camera/camera_info:=camera_info</remapping>
+              <remapping>camera/depth/camera_info:=depth/camera_info</remapping>
+              <remapping>camera/points:=depth/points</remapping>
+            </ros>
+            <camera_name>${name}</camera_name>
+            <frameName>${name}_link</frameName>
+            <hack_baseline>0.07</hack_baseline>
+            <min_depth>0.05</min_depth>
+            <max_depth>8.0</max_depth>
+          </plugin>
+        </sensor>
+      </xacro:unless>
     </gazebo>
   </xacro:macro>

File: simrobo_description/urdf/sensors/camera.urdf.xacro (robot description, xacro)
@@ -2,5 +2,5 @@
 <robot name="camera" xmlns:xacro="http://www.ros.org/wiki/xacro">
   <xacro:include filename="$(find simrobo_description)/urdf/sensors/camera.gazebo.xacro"/>
-  <xacro:macro name="camera" params="name depth width height mass parent *origin">
+  <xacro:macro name="camera" params="name use_ignition:=true depth width height mass parent *origin">
     <material name="${name}_color">
       <color rgba="0.70196 0.70196 0.70196 1.0"/>
@@ -34,5 +34,5 @@
     </joint>
     <!-- Gazebo Plugin -->
-    <xacro:camera_gazebo name="${name}"/>
+    <xacro:camera_gazebo name="${name}" use_ignition="${use_ignition}"/>
   </xacro:macro>
 </robot>

File: simrobo_description/urdf/simrobo.urdf.xacro (robot description, xacro)
@@ -8,6 +8,6 @@
   <xacro:include filename="$(find simrobo_description)/urdf/sensors/velodyne.urdf.xacro" />
   <!--xacro:include filename="$(find simrobo_description)/urdf/sensors/imu.urdf.xacro" />
-  <xacro:include filename="$(find simrobo_description)/urdf/sensors/gps.urdf.xacro" />
-  <xacro:include filename="$(find simrobo_description)/urdf/sensors/camera.urdf.xacro" / -->
+  <xacro:include filename="$(find simrobo_description)/urdf/sensors/gps.urdf.xacro" / -->
+  <xacro:include filename="$(find simrobo_description)/urdf/sensors/camera.urdf.xacro" />
   <xacro:include filename="$(find simrobo_description)/urdf/simrobo.ros2_control.xacro" />
   <!-- arg -->
@@ -108,8 +108,8 @@
   <xacro:gps name="gps" parent="base_link" length="${gps_length}" height="${gps_height}" mass="${gps_mass}">
     <origin xyz="0 0 ${body_height/3}" rpy="0 0 0"/>
-  </xacro:gps>
-  <xacro:camera name="camera" parent="base_link" depth="${camera_depth}" width="${camera_width}" height="${camera_height}" mass="${camera_mass}">
+  </xacro:gps -->
+  <xacro:camera name="camera" use_ignition="${use_ignition}" parent="base_link" depth="${camera_depth}" width="${camera_width}" height="${camera_height}" mass="${camera_mass}">
     <origin xyz="${(body_depth+camera_depth)/2} 0 ${camera_pos_z}" rpy="0 0 0"/>
-  </xacro:camera -->
+  </xacro:camera>
   <!-- ======== ros2_control ======== -->
   <xacro:simrobo_ros2_control name="simrobo" use_ignition="${use_ignition}"/>
